File: hardware/pcb/katanori61_voice/katanori61_voice.kicad_sch (KiCad schematic)
At the start: 214 parts, among them J10 BAT (JST-PH), J13 USB-C, J15 MIC RISER, J2 OLED, J5 SPK OUT, J6 BTN2, J7 REED+TOGGLE, Q1 MMUN2133LT1G, Q103 LBSS138WT1G, Q104 S9013W, U1 TPS61090RSAR, U102 XU316-1024-QF60B-C32, U103 W25Q32JVSSIQ, U106 SN74LVC125APWR, U108 TLV320AIC3204IRHBR, U109 TPA6211A1DGNR, U110 TPS62827DMQR, U111 ME6211C18M5G-N, U112 TPS62065DSGR, U118 SGM2036S-3.3XXDH4G/TR, U2 MCP73871-2CCI/ML, U3 INA226AIDGSR, U4 AS5600-ASOM, U5 ESP32-S3-WROOM-1U-N16R8, X101 24MHz 12pF

Commit message: 足形: Voice PE の板から voicepe.pretty（26 種）を起こす
置かれた足形（大半が裏面・回転つき）を、表向き・回転 0 のライブラリの形へ戻した。
検算: 元と同じ面・回転で置き直すと 171 部品の全パッドが位置・向き・層で一致。
QFN・TSSOP・SOIC・SOT-23-5・マイクの 1 番ピンは上から見て反時計回り。
C0603・R0603 は同じ名前で 2 通りのパッドがあったので、2 つ目を _v2 に分けた。
Parts:
- C122, C123: footprint voicepe:C0603 -> voicepe:C0603_v2
- R199, R200: footprint voicepe:R0603 -> voicepe:R0603_v2
Changed lines of the file:
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@@
 			)
 		)
-		(property "Footprint" "voicepe:C0603"
+		(property "Footprint" "voicepe:C0603_v2"
 			(at 647.70 165.10 0)
 			(effects
@@
 			)
 		)
-		(property "Footprint" "voicepe:C0603"
+		(property "Footprint" "voicepe:C0603_v2"
 			(at 660.40 167.64 0)
 			(effects
@@
 			)
 		)
-		(property "Footprint" "voicepe:R0603"
+		(property "Footprint" "voicepe:R0603_v2"
 			(at 571.50 193.04 0)
 			(effects
@@
 			)
 		)
-		(property "Footprint" "voicepe:R0603"
+		(property "Footprint" "voicepe:R0603_v2"
 			(at 612.14 193.04 0)
 			(effects

Commit message: 統合基板: JTAG をテストパッドに・多角形パッド・自動配線 5 回目（15 パス・ネックダウン無し）
- J105（20 ピン）を外し、XU316 のそばに 2×4 のテストパッド J16 を置く
- DSN: 回ったパッド・多角形のパッドを凸包の多角形で渡す（U118 の間隔違反が消えた）
- route.py: 板ごとに Freerouting の設定を明示（CLI の設定が全体の設定ファイルに残るため）
- 結果: 未配線 6 ネット（U102 の水晶・PLL・I2S の周りだけ）、R46/ESP_EN の間隔 0.1147 が 3 件
- gen_sch_voice / gen_pcb_voice には次の段（受動部品を 0402/0603 に・線 0.2 すきま 0.15）の
  コードも入っているが、この出力はその前の規則で作った物
Parts:
- removed J105: ~, voicepe:JTAG_2X10_1.27_SMD, symbol Seeed_libdb:Connector/1.27Header
- removed Q104: S9013W, voicepe:SOT-323, symbol Seeed_libdb:Transistor/305010001
- removed R128: 470K, voicepe:R0402, symbol Seeed_libdb:Resistors/301010069
- removed R132, R133: 22R, voicepe:R0402, symbol Seeed_libdb:Resistors/301010002
- added C112: 100nF, voicepe:C0402, symbol Seeed_libadl:Capacitors/302010024
- added C210: 1uF, voicepe:C0402, symbol Seeed_libdb:Capacitors/302013249
- added J16: XU316 JTAG, katanori:JTAG_TP_2x4_P2.54mm, symbol Connector_Generic:Conn_02x04_Odd_Even
- Q104: renamed from C210; value 1uF -> S9013W; footprint voicepe:C0402 -> voicepe:SOT-323; symbol Seeed_libdb:Capacitors/302013249 -> Seeed_libdb:Transistor/305010001; LCSC (none) -> C2919788; Note Voice PE C110（XMOS） -> Voice PE Q4（XMOS）
- R128: renamed from C112; value 100nF -> 470K; footprint voicepe:C0402 -> voicepe:R0402; symbol Seeed_libadl:Capacitors/302010024 -> Seeed_libdb:Resistors/301010069; Note Voice PE C12（XMOS） -> Voice PE R28（XMOS）
Connections:
- net GND: now also C112.2, C210.2, J16.7 (Pin_7); no longer R128.2
- net N_Q104_B: now also Q104.1 (B)
- net N_Q104_C: now also Q104.3 (C), R128.1
- net RST_N: now also J16.6 (Pin_6)
- net TCK: now also J16.3 (Pin_3)
- net TDI: now also J16.4 (Pin_4)
- net TDO: now also J16.5 (Pin_5)
- net TMS: now also J16.2 (Pin_2)
- net V18: now also J16.1 (Pin_1)
- net V5: now also R128.2
- net VDD_MIC: now also C112.1, C210.1; no longer Q104.1, R128.1
- net N_U102_X1D18: no longer names the net of U102.36 (X1D18)
- net N_U102_X1D19: no longer names the net of U102.37 (X1D19)
- net XL_DN0: no longer names the net of U102.35 (X1D17)
- net XL_DN1: no longer names the net of U102.33 (X1D16)
- no-connect marks 40 -> 44
Other:
- moved on the sheet: R128
