File: hardware/pcb/katanori61/katanori61.kicad_sch (KiCad schematic)
At the start: 55 parts, among them J1 XIAO RISER, J10 BAT (JST-PH), J13 USB-C, J2 OLED, J4 SPK IN, J5 SPK OUT, J6 BTN2, J7 REED+TOGGLE, K31 G6S-2F DC5, Q1 MMUN2133LT1G, Q2 AO3401A, Q31 SS8050, U1 TPS61090RSAR, U2 MCP73871-2CCI/ML, U3 INA226AIDGSR, U4 AS5600-ASOM

Commit message: pcb v6.1: J4 と J6 を縦の B2B-PH-K へ・J10 の極性を「手前が ＋ ・奥が GND」に戻す
🔒 ユーザー 2026-09-16 夕「J4とJ6を縦にして、J10の極性も手前奥に戻して」。

■ なぜ縦にしたか
J4（SPK IN）と J6（BTN2）は横出しで、抜く向きが**盤面の内側**（J4 は +Y・J6 は −Y）だった。
挿したプラグの胴が板の上へ 2.0 出るので、J4 は板の Y 14.30〜16.30、J6 は Y 21.20〜22.70 を塞ぐ。
gen_pcb の警告でも J4 の指の所に J13、J6 の指の所に R6・R7・D31・Q31・J1（背 8.5）が居て、
さらに「J6 の通り道が電池の下（挿し直すには電池を外す）」が出ていた。縦にすると全部消える。
筐体側は 56 個の模型でも plugpath が空で、殻は邪魔していない（別セッションが確認済み）。

■ J10 の極性が戻った
J10 のパッドを X 並びにしていたのは、J4 に挿さったプラグ（Y 14.30〜16.30）と
USB-C のシェルの足（20.63〜）に挟まれて 4.33 しか無く、6.9 の枠が入らなかったため。
J4 が縦になってその帯が消えたので **Y 並びへ戻した**。
  1 番 GND  → 板 (75.700, 16.950) ＝ 奥（ハッチ側）
  2 番 VBAT ＋ → 板 (75.700, 14.950) ＝ 手前（OLED 側）
PowerBoost B1 と同じ言い方に戻ったので、2026-09-16 夕に「左／右」で書き直した手順は
もう一度「手前／奥」に戻る。docs/PCB-V61.md 8 章を直した。

■ 置き直した枠（板の座標）
  J4  X 71.850〜78.750 / Y  6.250〜11.750（旧 Y 6.20〜14.80）。パッドは Y 8.45
      ⚠ 芯の Y は 9.00。8.60 だと枠の前端が取付穴 (72.5, 3.5) のナット（半径 2.56）へ 0.21 入る
  J6  X 14.050〜20.950 / Y 27.250〜32.750（旧 Y 22.70〜31.30）
  J10 X 73.500〜79.000 / Y 12.500〜19.400（旧 X 73.00〜79.90 / Y 14.475〜19.975）
      足は J4 の胴（Y 〜11.75）から 2.6・枠は USB-C の足（20.63）から 1.23

■ 足形は回路図が持っている
gen_pcb.py の BOX_PLACE だけ替えても足形は変わらない（place_footprint はネットリストの fp を使う）。
gen_sch.py の FP_PORT["PHIN"] と J6 の part() も B2B-PH-K へ替えること。
SPK OUT（J5）は口が板の**左の縁**（−X）を向いていて盤面を食わないので横出しのまま。
板の面に沿ってプラグが入るのは J5 だけになったので、gen_pcb の CONN も J5 だけにした。

■ 検査
回路図 0 件 / パッドの位置 11 点一致 / 重なり 0 / プラグの通り道 1 口すべて空き
DRC エラー 0・未接続 0・回路図との食い違い 0 / 銅箔のすきま 下回り 0 件（最小 0.151）
check_fab「奥（Y 16.95）が GND ／ 手前（Y 14.95）が VBAT」/ 地図の重なり なし
筐体 16 項目すべて期待値（hit_wires は 2.75 → 2.74）
STL 7 点 preflight: 中身 1 個・二重面 0・**🔴 0**（蓋の 0.22mm は 9072479 で解消済み）

■ 筐体側
pcb/v61_parts.scad を作り直した（gen_case_parts.py の PORTS も J4・J6 を上向きへ）。
SPK IN の線は「横から寄せて上から降ろす」形に引き直し。走る高さを
「嵌合したプラグの頭の 2.0 上」にした（旧 zl は横出しの背 4.8 を足した数で、縦の胴 6.0 ＋ 嵌合 2.0 より低く、プラグの頭を貫く）。
Parts:
- J4: footprint Connector_JST:JST_PH_S2B-PH-K_1x02_P2.00mm_Horizontal -> Connector_JST:JST_PH_B2B-PH-K_1x02_P2.00mm_Vertical
- J6: footprint Connector_JST:JST_PH_S2B-PH-K_1x02_P2.00mm_Horizontal -> Connector_JST:JST_PH_B2B-PH-K_1x02_P2.00mm_Vertical; Note 天板の会話ボタンへ 2 本 -> 天板の会話ボタンへ 2 本。⭐ 2026-09-16 夕に横出し → **縦**（🔒 ユーザー「J4とJ6を縦にして」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
Changed lines of the file:
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@@
 			)
 		)
-		(property "Footprint" "Connector_JST:JST_PH_S2B-PH-K_1x02_P2.00mm_Horizontal"
+		(property "Footprint" "Connector_JST:JST_PH_B2B-PH-K_1x02_P2.00mm_Vertical"
 			(at 30.48 243.84 0)
 			(effects
@@
 			)
 		)
-		(property "Footprint" "Connector_JST:JST_PH_S2B-PH-K_1x02_P2.00mm_Horizontal"
+		(property "Footprint" "Connector_JST:JST_PH_B2B-PH-K_1x02_P2.00mm_Vertical"
 			(at 109.22 243.84 0)
 			(effects
@@
 			)
 		)
-		(property "Note" "天板の会話ボタンへ 2 本"
+		(property "Note" "天板の会話ボタンへ 2 本。⭐ 2026-09-16 夕に横出し → **縦**（🔒 ユーザー「J4とJ6を縦にして」）。横出しは −Y（盤面の内側）で、指の所に J1（背 8.5 のライザー）が居て、通り道が電池の下にも当たっていた"
 			(at 109.22 243.84 0)
 			(effects

Commit message: pcb v6.1: 電源部を電流の順に並べ直す（電池の道 217 → 11.4 mΩ・INA226 のケルビン成立）
電源部は旧 PowerBoost 基板 → v6 → v6.1 の**二重の写し**で置かれていて、
v6.1 の板の上で並べた人がいなかった（gen_pcb.py の写しの注「ここで並べ直して
はいない」のまま）。その結果:

  ・電池の口 J10（板 X 76）からシャント R41（X 30）まで電流が板を横断し、
    自動配線の既定 0.2mm のままで配線 107mm ＝ 217mΩ
  ・シャント R41 と電流計 U3 が 23mm 離れ、センス線が R41 のパッドではなく
    11.9mΩ 手前（Q2 の足元）と 73.7mΩ 先（U2 の VBAT）から出ていた。
    INA226 は 10mΩ ではなく 96.7mΩ ＝ **9.7 倍**を見ていた
  ・USB-C J13 から充電 IC U2 まで 52mm

v5 で正しく読めていたのは、INA226 モジュールの上でシャントと IC が数 mm しか
離れておらず、ケルビンがモジュールの中で取れていたからである。v6.1 でシャントを
板に降ろしたときに、回路図（同じネット）は写ったが置き方（同じ点）が写らなかった。

並べ直し（板の座標で明示・写しをやめた）:
  J10 電池 → Q2 逆接保護 → R41 シャント → U2 充電 → L1・U1 昇圧 → J1 XIAO
  U3 は R41 の真上。USB-C は U2 のすぐ前の縁へ。

  電池の道      107mm 217.2mΩ → 13.7mm 11.4mΩ（充電 560mA で 6.4mV・1A で 11.4mV）
  R41 → U3      23.2mm → 3.0mm
  J13 → U2      52.0mm → 12.9mm
  ホットループ  7.4mm → 3.3mm（U1 を 180° 回して SW を L1 の側へ）
  SW            6.2mm → 4.6mm

入れた仕組み:
  ・dsn.py    ネットの組ごとの線幅（電池 0.6 / VSYS・SW・V5 0.4 / VBUS 0.2）
  ・gen_pcb.py PRE_TRACKS … 先に手で引いて固定する線。R41 のケルビン 2 本。
               ep_vias()  … U1・U2 の放熱パッドに GND ビア 4 本ずつ（配置から計算）
  ・route.py  locked の線と穴を merge で残し、SES に返る protect の写しは捨てる
  ・gen_sch.py R41 に「ケルビン必須・PRE_TRACKS を見よ」と経緯ごと残した

ついでに直したもの:
  ・USB-C を動かしたのに VBUS のベタが板の右端に残っていた（isolated_copper）。
    口の向きに追従させた
  ・Freerouting の最適化の段が、配線の段より悪い版から始めて書き出す（未接続 1 → 6）。
    統合基板で 2026-09-15 に見たのと同じ不具合。v6.1 側でも切った

検算: 未接続 0 ／ 回路図との差 0 ／ DRC エラー 0 ／ 銅のすきま 下回り 0。
ケルビンは「負荷の道 ＋ センス線 ＝ 直に測った値」の一致で成立を確認した。

残る警告: silk_over_copper 2 件（U1・U2 のシルクの角が隣のパッドに 0.1 乗る。
逃がすと未接続が 2 本出たので警告を取った）。lib_footprint_issues 59 件と
silk_edge_clearance 2 件は以前からあるもの。
Parts:
- R41: Note シャント 10mΩ（今のモジュールと同じ値） -> シャント 10mΩ（今のモジュールと同じ値）。🔴 ケルビン必須 — gen_pcb.py の PRE_TRACKS を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
Changed lines of the file:
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@@
 			)
 		)
-		(property "Note" "シャント 10mΩ（今のモジュールと同じ値）"
+		(property "Note" "シャント 10mΩ（今のモジュールと同じ値）。🔴 ケルビン必須 — gen_pcb.py の PRE_TRACKS を見よ"
 			(at 261.62 40.64 0)
 			(effects

Commit message: pcb v6.1: R2・R6・R7 を 0603 へ／V5 を 0.8mm の独立した組へ／手はんだの GND にサーマル
外からの指摘 4 件のうち 1〜4 を直す。

1. 足形の食い違い
   Basic で選び直した R2(C23137)・R6(C22961)・R7(C23254) は 0603 なのに
   足形が 0805 のままだった。0805 のパッドの内側の間 0.875 に 0603 の胴 1.6 が
   両端 0.36 ずつ乗るだけで、機械実装で着かないか立つ。

3. V5 が内層を遠回り
   U1 → J1（XIAO）が 57.49mm、うち 57.3mm が In2.Cu。JLCPCB の 4 層は
   内層 0.5oz が既定なので、同じ幅でも抵抗が 2 倍になる。
   0.4mm → 0.8mm の独立した組にして 29.46mm・18.1mΩ（前 141.5mΩ）。
   0.3A で 5.4mV（前 42.5mV）。

4. 電池の道の数字が古い
   gen_pcb.py の「12mm・10mΩ」は J10 を板の真ん中に置いていたときの値。
   実測に入れ替え: J10→Q2 31.16mm/25.5mΩ、Q2→R41 2.18mm/1.8mΩ、
   R41→U2 3.63mm/3.0mΩ、計 36.97mm・30.3mΩ（1A で 30mV）。

2. GND ベタが全パッド直結
   4 層で In1 が全面 GND になり、手はんだの口は 3 層が足に直結してこてで
   温度が逃げる。HAND_SOLDER の貫通 GND だけ thermal relief にした
   （J1-2 / J2-1 / J6-1 / J7-2 / J7-4 / J10-1 の 6 本）。表面実装は直結のまま。
   細いパッドは spoke が 1 本しか立たないので katanori61.kicad_dru を生成し、
   貫通パッドだけ min_resolved_spokes 1 に緩める。

ついでに見つけた不具合
   pad_box() が部品の角度を足しておらず、270° 置きの U3 で縦横が入れ替わって
   いた。ケルビンの線の端が U3 のパッドの 0.335 外に落ちていたのを自動配線が
   繕っていた。
   fab.py の JLC_ROT に R_0603_1608Metric（2 本足・補正 0）を足した。
   gen_case_parts.py の「いまの手書きの表は 9 個」は表を生成に変えた時点で
   嘘になっていたので消した。

検算
   配線 708 本・貫通穴 59 個・未接続 0・回路図との差 0・DRC エラー 0
   （警告は留め穴 4 と USB-C のシルク 2 のみ。starved_thermal は 0）
   模型・STL・ガーバー・BOM・CPL を出し直した。
   レジンの sk_hub 12.02mm³ は以前からの当たり（HEAD で 12.59）。
Parts:
- R2, R6, R7: footprint Resistor_SMD:R_0805_2012Metric -> Resistor_SMD:R_0603_1608Metric
Changed lines of the file:
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@@
 			)
 		)
-		(property "Footprint" "Resistor_SMD:R_0805_2012Metric"
+		(property "Footprint" "Resistor_SMD:R_0603_1608Metric"
 			(at 160.02 40.64 0)
 			(effects
@@
 			)
 		)
-		(property "Footprint" "Resistor_SMD:R_0805_2012Metric"
+		(property "Footprint" "Resistor_SMD:R_0603_1608Metric"
 			(at 93.98 132.08 0)
 			(effects
@@
 			)
 		)
-		(property "Footprint" "Resistor_SMD:R_0805_2012Metric"
+		(property "Footprint" "Resistor_SMD:R_0603_1608Metric"
 			(at 104.14 132.08 0)
 			(effects

Commit message: pcb v6.1: VBUS の最後の枝を太く（C8 を U2 の入力ピンの真上へ）／電源のコンデンサの横に GND の穴
発注前レビューで出た 1 件。幹（J13 → C8）は 0.6mm にしてあったが、C8 → U2 の 18・19 番は
「3mm の枝」のつもりで自動配線任せで、板を測ると B.Cu 0.2mm × 3.3mm → 穴 → F.Cu 0.2mm × 2.7mm
＋ ピンの足 0.66 ＝ 6.6mm・16mΩ。太くした幹（15.2mm・12.5mΩ）より大きかった。
原因は線幅ではなく配置:
  ・C8 が横向きで、2 番（GND）の下端と U2 のピン列のあいだが 0.66mm
  ・C8 の 2 番が乗る表の GND の島に穴が無く、GND の 0.2mm 線が C8 の 1 番の真下を横切る

直し:
  ・C8 を縦（90°）にして 1 番を U2 の 17〜19 番（3 本とも VBUS）の真上へ。1 番 → ピンは 1.2mm
    隣の 20 番（VSYS）・16 番（VLIPO）まで 0.275 ずつ。幹は 1 番の左の横で表へ上がる
  ・C41 34.0 → 36.4・R13 23.0 → 23.5（C8 の置き場と GND の穴の分）
  ・cap_gnd_vias(): C8・C6・C9・C1 の GND パッドの横に GND の穴（📄 TPS61090 12.1）
    C2 は置ける側が無いので外した（下は V5 の幹・上は R4 の FB まで 0.18・右は C6 の V5 まで 0.15）
  ・check_pre(): 先に引いた穴 × 別ネットの先に引いた線。最初の置き方で GND の穴が裏の
    VBUS の幹と V5 の幹に乗った（protect どうしなので DRC まで出ない短絡）。生成で止める

結果（板から測った値・外層 1oz）: J13 → U2 の入力 28.5 → 13.4mΩ・全区間 0.6mm 以上・穴 2 個。
DRC エラー 0・未接続 0（警告は前からの 6 件）。check_pcb 0 件（最小 VSYS ↔ LBO 0.151）。
check_sch 0 件。check_fab 合わない所なし。ガーバー・BOM・CPL・v61_parts を出し直した。
⚠ 筐体側の当たり検査（case_v6_1.scad）は回していない。動いたのは背 0.45〜1.25 の 0805 が 3 個。

古い記述の片付け:
  ・CHECK_PADS の Q2 が 1.0 古く、生成のたびに警告が 3 行出ていた（向きは合っていた）
  ・gen_pcb.py 頭の「J10 → Q2 28.6mm 23.9mΩ」→ 37.6mm 32mΩ（AS5600 をよけて回す前の値だった）
  ・PCB-V61.md 4.1 のシルク 0.12 の ⬜（ガーバーは表裏とも 0.150 だけ）・5 章に --incremental の件
  ・gen_sch.py の J13 の注記（1.53 出し → 1.3）
Parts:
- J13: Note 充電の口。D+/D− と SBU は使わない。v6.1 は板の縁から 1.53 しか出ないので前のシェルの足 2 本も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 -> 充電の口。D+/D− と SBU は使わない。v6.1 は板の後ろの縁から 1.3 出し（⭐ 2026-09-17）で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
Changed lines of the file:
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@@
 			)
 		)
-		(property "Note" "充電の口。D+/D− と SBU は使わない。v6.1 は板の縁から 1.53 しか出ないので前のシェルの足 2 本も板に載る"
+		(property "Note" "充電の口。D+/D− と SBU は使わない。v6.1 は板の後ろの縁から 1.3 出し（⭐ 2026-09-17）で、シェルの足 4 本とも板に載る"
 			(at 347.98 50.80 0)
 			(effects

Commit message: pcb v6.1: CPL の向きと位置を JLCPCB の品番ごとの足形（EasyEDA）から出す／Q1 を足形のある YTL C53477467 へ
- 公開の補正表（JLCKicadTools）を足形の名前で当てるのをやめ、品番の足形を KiCad の足形に重ねて角度と原点のずれを出す（jlc_fp.py）。
  表の値では U1・Q2・Q31・K31・J13 が 90°／180° 回って載り、K31 は 1.27・J13 は 1.57 ずれていた
- check_fab.py に別の道の検算: CPL どおりに JLCPCB の足形を置き、IPC-D-356 のパッド・穴に乗るかを見る（48 個・最大 0.28）
- 足形の無い品番では fab.py が止まる。「プレビューで見る」で逃がさない
- Q1: CBI C21714196 は EasyEDA に足形が無く、JLCPCB のプレビューでも市松模様の印しか出ない。
  電気的に同じ（4.7k/47k）YTL C53477467 へ。JLCPCB のプレビューで極性のある部品を全部目で見て合っていた
Parts:
- Q1: LCSC C21714196 -> C53477467
Changed lines of the file:
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@@
 			)
 		)
-		(property "LCSC" "C21714196"
+		(property "LCSC" "C53477467"
 			(at 33.02 91.44 0)
 			(effects
